File: Schematics/EchoHand_v2/EchoHand_v2.kicad_sch (KiCad schematic)
At the start: 2 parts, among them M1 Motor_Servo, U1 ESP32-WROOM-32D

Commit message: Upload release candidate schematic
Parts:
- removed M1: Motor_Servo, symbol Motor:Motor_Servo
- removed U1: ESP32-WROOM-32D, RF_Module:ESP32-WROOM-32D, symbol RF_Module:ESP32-WROOM-32D
- added C1: C_Polarized, symbol Device:C_Polarized
- added J1: Screw_Terminal_01x02, symbol Connector:Screw_Terminal_01x02
- added J10, J11, J2, J3, J4, J5, J6, J7, J8, J9: Conn_01x03_Socket, symbol Connector:Conn_01x03_Socket
- added U1: ESP32-S3, Package_DFN_QFN:QFN-56-1EP_7x7mm_P0.4mm_EP4x4mm, symbol MCU_Espressif:ESP32-S3
- added U2: HC-05, HC-05:XCVR_HC-05, symbol HC-05:HC-05
Connections:
- net +5V: now also C1.1, J1.2 (Pin_2), J10.2 (Pin_2), J11.2 (Pin_2), J7.2 (Pin_2), J8.2 (Pin_2), J9.2 (Pin_2)
- net GND: now also C1.2, J1.1 (Pin_1), J10.3 (Pin_3), J11.3 (Pin_3), J2.3 (Pin_3), J3.3 (Pin_3), J4.3 (Pin_3), J5.3 (Pin_3), J6.3 (Pin_3), J7.3 (Pin_3), J8.3 (Pin_3), J9.3 (Pin_3), U1.57 (GND), U2.13 (GND), U2.21 (GND), U2.22 (GND)
- new net +3V3: J2.1 (Pin_1), J3.1 (Pin_1), J4.1 (Pin_1), J5.1 (Pin_1), J6.1 (Pin_1), U1.2 (VDD3P3), U1.20 (VDD3P3_RTC), U1.29 (VDD_SPI), U1.3 (VDD3P3), U1.46 (VDD3P3_CPU), U1.55 (VDDA), U1.56 (VDDA), U2.12 (3.3_VCC)
- new net a_button: U1.17 (GPIO12)
- new net b_button: U1.18 (GPIO13)
- new net bluetooth_rx: U1.24 (GPIO18), U2.2 (UART-RX)
- new net bluetooth_tx: U1.23 (GPIO17), U2.1 (UART-TX)
- new net index_pot: J3.2 (Pin_2), U1.9 (GPIO4)
- new net index_servo: J8.1 (Pin_1), U1.40 (GPIO35)
- new net joystick_button: U1.16 (GPIO11)
- new net joystick_x: U1.14 (GPIO9)
- new net joystick_y: U1.15 (GPIO10)
- new net middle_pot: J4.2 (Pin_2), U1.12 (GPIO7)
- new net middle_servo: J9.1 (Pin_1), U1.41 (GPIO36)
- new net pinky_pot: J6.2 (Pin_2), U1.11 (GPIO6)
- new net pinky_servo: J11.1 (Pin_1), U1.43 (GPIO38)
- new net ring_pot: J5.2 (Pin_2), U1.10 (GPIO5)
- new net ring_servo: J10.1 (Pin_1), U1.42 (GPIO37)
- new net thumb_pot: J2.2 (Pin_2), U1.13 (GPIO8)
- new net thumb_servo: J7.1 (Pin_1), U1.51 (GPIO45)
Other:
- company: (none) -> University of Florida
- title: EchoHand -> EchoHand PCB
